File: matrix-flower-1/matrix-flower-1.kicad_sch (KiCad schematic)
At the start: 10 parts, among them U1 ATmega328P-A, Y1 Resonator_Small

Commit message: Update component information.
Parts:
- PWR1: now not fitted
Changed lines of the file:
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@@
 			)
 		)
-		(property "Datasheet" "~"
+		(property "Datasheet" "https://www.amazon.com/dp/B09GP9S1W7"
 			(at 179.07 105.41 0)
 			(effects
@@
 		(in_bom yes)
 		(on_board yes)
-		(dnp no)
+		(dnp yes)
 		(fields_autoplaced yes)
 		(property "Reference" "PWR1"
@@
 			)
 		)
-		(property "Datasheet" "~"
+		(property "Datasheet" "https://www.amazon.com/dp/B0BKSNMCV4"
 			(at 182.88 74.93 0)
 			(effects
